File: dev_board/dev_board.kicad_pcb (KiCad board)
At the start: 2 copper layers, 6 parts, among them J2 Left, J3 Right

Commit message: f
Parts:
- added C1: 2.2uF, Capacitor_SMD:C_0805_2012Metric, F.Cu at (60.5, 69.0)
- added C10: 100nF, Capacitor_SMD:C_0805_2012Metric, F.Cu at (82.2, 72.6)
- added C2: 2.2uF, Capacitor_SMD:C_0805_2012Metric, F.Cu at (62.5, 76.0)
- added C3: 4.7uF, Capacitor_SMD:C_0805_2012Metric, F.Cu at (82.2, 57.5)
- added C4: 1uF, Capacitor_SMD:C_0805_2012Metric, F.Cu at (52.5, 66.5)
- added C5: 100nF, Capacitor_SMD:C_0805_2012Metric, F.Cu at (52.5, 69.5)
- added C6: 100nF, Capacitor_SMD:C_0805_2012Metric, F.Cu at (82.2, 60.6)
- added C7: 100nF, Capacitor_SMD:C_0805_2012Metric, F.Cu at (82.2, 63.6)
- added C8: 1uF, Capacitor_SMD:C_0805_2012Metric, F.Cu at (82.2, 66.6)
- added C9: 100nF, Capacitor_SMD:C_0805_2012Metric, F.Cu at (82.2, 69.6)
- added J4: Conn_ARM_SWD_TagConnect_TC2030-NL, Connector:Tag-Connect_TC2030-IDC-NL_2x03_P1.27mm_Vertical, F.Cu at (88.5, 79.4)
- added J5: Conn_ARM_SWD_TagConnect_TC2030-NL, Connector:Tag-Connect_TC2030-IDC-NL_2x03_P1.27mm_Vertical, F.Cu at (70.0, 104.5)
- added Q1: BUT11, Package_TO_SOT_THT:TO-220-3_Vertical, F.Cu at (74.4, 95.0)
- added U1: nRF52810-QCxx, Package_DFN_QFN:QFN-32-1EP_5x5mm_P0.5mm_EP3.6x3.6mm, F.Cu at (121.0, 97.0)
- added U2: STM32H533CETx, Package_QFP:LQFP-48_7x7mm_P0.5mm, F.Cu at (120.5, 82.5)
- added U3: FT230XQ, Package_DFN_QFN:QFN-16-1EP_4x4mm_P0.65mm_EP2.1x2.1mm, F.Cu at (57.2, 113.4)
- added U3: FT232BM, Package_QFP:LQFP-32_7x7mm_P0.8mm, F.Cu at (120.0, 114.0)
- added U4: LT1963AxST-3.3, Package_TO_SOT_SMD:SOT-223-3_TabPin2, F.Cu at (51.0, 95.0)
Connections:
- J2 pad 1: +5V -> unconnected-(J2-Pin_1-Pad1)
- J2 pad 10: /PD10 -> unconnected-(J2-Pin_10-Pad10)
- J2 pad 11: /PD13 -> unconnected-(J2-Pin_11-Pad11)
- J2 pad 12: /PD12 -> unconnected-(J2-Pin_12-Pad12)
- J2 pad 13: /PD15 -> unconnected-(J2-Pin_13-Pad13)
- J2 pad 14: /PD14 -> unconnected-(J2-Pin_14-Pad14)
- J2 pad 15: /PC7 -> unconnected-(J2-Pin_15-Pad15)
- J2 pad 16: /PC6 -> unconnected-(J2-Pin_16-Pad16)
- J2 pad 17: /PC9 -> unconnected-(J2-Pin_17-Pad17)
- J2 pad 18: /PC8 -> unconnected-(J2-Pin_18-Pad18)
- J2 pad 19: /PA9_TX1 -> unconnected-(J2-Pin_19-Pad19)
- J2 pad 2: +5V -> unconnected-(J2-Pin_2-Pad2)
- J2 pad 20: /PA8 -> unconnected-(J2-Pin_20-Pad20)
- J2 pad 21: /PA11_USB_DM -> unconnected-(J2-Pin_21-Pad21)
- J2 pad 22: /PA10_RX1 -> unconnected-(J2-Pin_22-Pad22)
- J2 pad 23: /PA15 -> unconnected-(J2-Pin_23-Pad23)
- J2 pad 24: /PA12_USB_DP -> unconnected-(J2-Pin_24-Pad24)
- J2 pad 25: /PC11 -> unconnected-(J2-Pin_25-Pad25)
- J2 pad 26: /PC10 -> unconnected-(J2-Pin_26-Pad26)
- J2 pad 27: /PD0 -> unconnected-(J2-Pin_27-Pad27)
- J2 pad 28: /PC12 -> unconnected-(J2-Pin_28-Pad28)
- J2 pad 29: /PD2 -> unconnected-(J2-Pin_29-Pad29)
- J2 pad 3: +3.3V -> unconnected-(J2-Pin_3-Pad3)
- J2 pad 30: /PD1 -> unconnected-(J2-Pin_30-Pad30)
- J2 pad 31: /PD4 -> unconnected-(J2-Pin_31-Pad31)
- J2 pad 32: /PD3 -> unconnected-(J2-Pin_32-Pad32)
- J2 pad 33: /PD6 -> unconnected-(J2-Pin_33-Pad33)
- J2 pad 34: /PD5 -> unconnected-(J2-Pin_34-Pad34)
- J2 pad 35: /PB3 -> unconnected-(J2-Pin_35-Pad35)
- J2 pad 36: /PD7 -> unconnected-(J2-Pin_36-Pad36)
- J2 pad 37: /PB5 -> unconnected-(J2-Pin_37-Pad37)
- J2 pad 38: /PB4 -> unconnected-(J2-Pin_38-Pad38)
- J2 pad 39: /PB7 -> unconnected-(J2-Pin_39-Pad39)
- J2 pad 4: +3.3V -> unconnected-(J2-Pin_4-Pad4)
- J2 pad 40: /PB6 -> unconnected-(J2-Pin_40-Pad40)
- J2 pad 41: /PB9 -> unconnected-(J2-Pin_41-Pad41)
- J2 pad 42: /PB8 -> unconnected-(J2-Pin_42-Pad42)
- J2 pad 43: /PE1 -> unconnected-(J2-Pin_43-Pad43)
- J2 pad 44: /PE0 -> unconnected-(J2-Pin_44-Pad44)
- J2 pad 5: GND -> unconnected-(J2-Pin_5-Pad5)
- J2 pad 6: GND -> unconnected-(J2-Pin_6-Pad6)
- J2 pad 7: /PD9 -> unconnected-(J2-Pin_7-Pad7)
- J2 pad 8: /PD8 -> unconnected-(J2-Pin_8-Pad8)
- J2 pad 9: /PD11 -> unconnected-(J2-Pin_9-Pad9)
- J3 pad 1: +3.3V -> unconnected-(J3-Pin_1-Pad1)
- J3 pad 10: /PB12 -> unconnected-(J3-Pin_10-Pad10)
- J3 pad 11: /PB11 -> unconnected-(J3-Pin_11-Pad11)
- J3 pad 12: /PB10 -> unconnected-(J3-Pin_12-Pad12)
- J3 pad 13: /PE15 -> unconnected-(J3-Pin_13-Pad13)
- J3 pad 14: /PE14 -> unconnected-(J3-Pin_14-Pad14)
- J3 pad 15: /PE13 -> unconnected-(J3-Pin_15-Pad15)
- J3 pad 16: /PE12 -> unconnected-(J3-Pin_16-Pad16)
- J3 pad 17: /PE11 -> unconnected-(J3-Pin_17-Pad17)
- J3 pad 18: /PE10 -> unconnected-(J3-Pin_18-Pad18)
- J3 pad 19: /PE9 -> unconnected-(J3-Pin_19-Pad19)
- J3 pad 2: +3.3V -> unconnected-(J3-Pin_2-Pad2)
- J3 pad 20: /PE8 -> unconnected-(J3-Pin_20-Pad20)
- J3 pad 21: /PE7 -> unconnected-(J3-Pin_21-Pad21)
- J3 pad 22: /PB2 -> unconnected-(J3-Pin_22-Pad22)
- J3 pad 23: /PB1 -> unconnected-(J3-Pin_23-Pad23)
- J3 pad 24: /PB0 -> unconnected-(J3-Pin_24-Pad24)
- J3 pad 25: /PC5 -> unconnected-(J3-Pin_25-Pad25)
- J3 pad 26: /PC4 -> unconnected-(J3-Pin_26-Pad26)
- J3 pad 27: /PA7 -> unconnected-(J3-Pin_27-Pad27)
- J3 pad 28: /PA6 -> unconnected-(J3-Pin_28-Pad28)
- J3 pad 29: /PA5 -> unconnected-(J3-Pin_29-Pad29)
- J3 pad 3: GND -> unconnected-(J3-Pin_3-Pad3)
- J3 pad 30: /PA4 -> unconnected-(J3-Pin_30-Pad30)
- J3 pad 31: /PA3 -> unconnected-(J3-Pin_31-Pad31)
- J3 pad 32: /PA2 -> unconnected-(J3-Pin_32-Pad32)
- J3 pad 33: /PA1 -> unconnected-(J3-Pin_33-Pad33)
- J3 pad 34: /PA0 -> unconnected-(J3-Pin_34-Pad34)
- J3 pad 35: /PC3 -> unconnected-(J3-Pin_35-Pad35)
- J3 pad 36: /PC2 -> unconnected-(J3-Pin_36-Pad36)
- J3 pad 37: /PC1 -> unconnected-(J3-Pin_37-Pad37)
- J3 pad 38: /PC0 -> unconnected-(J3-Pin_38-Pad38)
- J3 pad 39: /PC13 -> unconnected-(J3-Pin_39-Pad39)
- J3 pad 4: GND -> unconnected-(J3-Pin_4-Pad4)
- J3 pad 40: /PE6 -> unconnected-(J3-Pin_40-Pad40)
- J3 pad 41: /PE5 -> unconnected-(J3-Pin_41-Pad41)
- J3 pad 42: /PE4 -> unconnected-(J3-Pin_42-Pad42)
- J3 pad 43: /PE3 -> unconnected-(J3-Pin_43-Pad43)
- J3 pad 44: /PE2 -> unconnected-(J3-Pin_44-Pad44)
- J3 pad 5: VDDA -> unconnected-(J3-Pin_5-Pad5)
- J3 pad 6: /VREF+ -> unconnected-(J3-Pin_6-Pad6)
- J3 pad 7: /PB15 -> unconnected-(J3-Pin_7-Pad7)
- J3 pad 8: /PB14 -> unconnected-(J3-Pin_8-Pad8)
- J3 pad 9: /PB13 -> unconnected-(J3-Pin_9-Pad9)
