File: dev_board/main_mcu.kicad_sch (KiCad schematic)
At the start: 3 parts, among them U2 STM32H533CETx

Commit message: f
Parts:
- added C10, C5, C6, C7, C9: 100nF, Capacitor_SMD:C_0805_2012Metric, symbol Device:C
- added C11: 0.1uF, symbol Device:C
- added C3: 4.7uF, Capacitor_SMD:C_0805_2012Metric, symbol Device:C
- added C4, C8: 1uF, Capacitor_SMD:C_0805_2012Metric, symbol Device:C
- added J4: Conn_ARM_SWD_TagConnect_TC2030-NL, Connector:Tag-Connect_TC2030-IDC-NL_2x03_P1.27mm_Vertical, symbol Connector:Conn_ARM_SWD_TagConnect_TC2030-NL
- added Q1: BUT11, Package_TO_SOT_THT:TO-220-3_Vertical, symbol Transistor_BJT:BUT11
- added SW1: SW_SPST, symbol Switch:SW_SPST
Connections:
- net GND: now also U2.23 (VSS), U2.35 (VSS), U2.47 (VSS), U2.8 (VSSA), C10.2, C11.2, C3.2, C4.2, C5.2, C6.2, C7.2, C8.2, C9.2, Q1.3 (E), SW1.2 (B); no longer C1.1, C2.2, U2.22 (VCAP), U2.46 (VCAP)
- net +BATT: now reaches U2.1 (VBAT)
- net +BATT: now also C4.1, C5.1
- net +3V3: now reaches U2.24 (VDD)
- net +3V3: now also U2.36 (VDD), U2.48 (VDD), U2.9 (VDDA), C10.1, C3.1, C6.1, C7.1, C8.1, C9.1, Q1.1 (B)
- net BOOT: now reaches U2.44 (BOOT0)
- net BOOT: now also Q1.2 (C)
- net RST: now reaches U2.7 (NRST)
- net RST: now also C11.1, J4.3 (~{RESET}), SW1.1 (A)
- new net: C2.2, U2.22 (VCAP)
- new net: C1.1, U2.46 (VCAP)
Other:
- note added: "Footprint too big consider switch to 0605"
- note added: "VBAT Charging Support"
- note removed: "Should Support VBAT"
- moved on the sheet: C1, C2
