File: dev_board/aux_mcu.kicad_sch (KiCad schematic)
At the start: 1 part, among them U1 nRF52810-QCxx

Commit message: f
Parts:
- added C12: 0.8pf, symbol Device:C
- added C13, C14: 12pF, symbol Device:C
- added C15: 100nF, symbol Device:C
- added C16: N.C., symbol Device:C
- added C17: 100pF, symbol Device:C
- added C18: 1uF, symbol Device:C
- added C19: 4.7uF, symbol Device:C
- added C20: 0.1uF, symbol Device:C
- added J5: Conn_ARM_SWD_TagConnect_TC2030-NL, Connector:Tag-Connect_TC2030-IDC-NL_2x03_P1.27mm_Vertical, symbol Connector:Conn_ARM_SWD_TagConnect_TC2030-NL
- added L1: 3.9nH, symbol Device:L
- added SW2: SW_SPST, symbol Switch:SW_SPST
- added Y1: Crystal, symbol Device:Crystal
Connections:
- net DET1: now reaches U1.1 (DEC1)
- net DET1: now also C15.1
- net RST1: now reaches U1.16 (P0.21/~{RESET})
- net RST1: now also C20.1, J5.3 (~{RESET}), SW2.1 (A)
- net at U1.19 (ANT): now also C12.1, L1.2
- net GND: now reaches U1.20 (VSS), U1.29 (VSS), U1.33 (VSS)
- net GND: now also C12.2, C13.2, C14.1, C15.2, C16.1, C17.1, C18.1, C19.2, C20.2, SW2.2 (B)
- net DET2: now reaches U1.21 (DEC2)
- net DET2: now also C16.2
- net DET3: now reaches U1.22 (DEC3)
- net DET3: now also C17.2
- net at U1.23 (XC1): now also C13.1, Y1.2
- net at U1.24 (XC2): now also C14.2, Y1.1
- net +3V3: now reaches U1.25 (VDD), U1.32 (VDD), U1.9 (VDD)
- net +3V3: now also C19.1
- net DET4: now reaches U1.30 (DEC4)
- net DET4: now also C18.2
- new net RF: L1.1
- no-connect marks 0 -> 1

Commit message: f
Parts:
- Y1: value Crystal -> 32MHz
Changed lines of the file:
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@@
 		(on_board yes)
 		(dnp no)
-		(fields_autoplaced yes)
 		(property "Reference" "Y1"
-			(at 114.3 104.1399 90)
+			(at 113.792 105.41 90)
 			(effects
 				(font
@@
 			)
 		)
-		(property "Value" "Crystal"
-			(at 114.3 106.6799 90)
+		(property "Value" "32MHz"
+			(at 112.014 108.966 90)
 			(effects
 				(font
