File: dev_board/dev_board.kicad_sch (KiCad schematic)
At the start: 6 parts, among them J2 Left, J3 Right

Commit message: f
Connections:
- removed net +3.3V: J2.3 (Pin_3), J2.4 (Pin_4), J3.1 (Pin_1), J3.2 (Pin_2)
- net +5V: no longer names the net of J2.1 (Pin_1)
- net +5V: no longer J2.2 (Pin_2)
- removed net GND: J2.5 (Pin_5), J2.6 (Pin_6), J3.3 (Pin_3), J3.4 (Pin_4)
- net PA0: no longer names the net of J3.34 (Pin_34)
- net PA1: no longer names the net of J3.33 (Pin_33)
- net PA10_RX1: no longer names the net of J2.22 (Pin_22)
- net PA11_USB_DM: no longer names the net of J2.21 (Pin_21)
- net PA12_USB_DP: no longer names the net of J2.24 (Pin_24)
- net PA15: no longer names the net of J2.23 (Pin_23)
- net PA2: no longer names the net of J3.32 (Pin_32)
- net PA3: no longer names the net of J3.31 (Pin_31)
- net PA4: no longer names the net of J3.30 (Pin_30)
- net PA5: no longer names the net of J3.29 (Pin_29)
- net PA6: no longer names the net of J3.28 (Pin_28)
- net PA7: no longer names the net of J3.27 (Pin_27)
- net PA8: no longer names the net of J2.20 (Pin_20)
- net PA9_TX1: no longer names the net of J2.19 (Pin_19)
- net PB0: no longer names the net of J3.24 (Pin_24)
- net PB1: no longer names the net of J3.23 (Pin_23)
- net PB10: no longer names the net of J3.12 (Pin_12)
- net PB11: no longer names the net of J3.11 (Pin_11)
- net PB12: no longer names the net of J3.10 (Pin_10)
- net PB13: no longer names the net of J3.9 (Pin_9)
- net PB14: no longer names the net of J3.8 (Pin_8)
- net PB15: no longer names the net of J3.7 (Pin_7)
- net PB2: no longer names the net of J3.22 (Pin_22)
- net PB3: no longer names the net of J2.35 (Pin_35)
- net PB4: no longer names the net of J2.38 (Pin_38)
- net PB5: no longer names the net of J2.37 (Pin_37)
- net PB6: no longer names the net of J2.40 (Pin_40)
- net PB7: no longer names the net of J2.39 (Pin_39)
- net PB8: no longer names the net of J2.42 (Pin_42)
- net PB9: no longer names the net of J2.41 (Pin_41)
- net PC0: no longer names the net of J3.38 (Pin_38)
- net PC1: no longer names the net of J3.37 (Pin_37)
- net PC10: no longer names the net of J2.26 (Pin_26)
- net PC11: no longer names the net of J2.25 (Pin_25)
- net PC12: no longer names the net of J2.28 (Pin_28)
- net PC13: no longer names the net of J3.39 (Pin_39)
- net PC2: no longer names the net of J3.36 (Pin_36)
- net PC3: no longer names the net of J3.35 (Pin_35)
- net PC4: no longer names the net of J3.26 (Pin_26)
- net PC5: no longer names the net of J3.25 (Pin_25)
- net PC6: no longer names the net of J2.16 (Pin_16)
- net PC7: no longer names the net of J2.15 (Pin_15)
- net PC8: no longer names the net of J2.18 (Pin_18)
- net PC9: no longer names the net of J2.17 (Pin_17)
- net PD0: no longer names the net of J2.27 (Pin_27)
- net PD1: no longer names the net of J2.30 (Pin_30)
- net PD10: no longer names the net of J2.10 (Pin_10)
- net PD11: no longer names the net of J2.9 (Pin_9)
- net PD12: no longer names the net of J2.12 (Pin_12)
- net PD13: no longer names the net of J2.11 (Pin_11)
- net PD14: no longer names the net of J2.14 (Pin_14)
- net PD15: no longer names the net of J2.13 (Pin_13)
- net PD2: no longer names the net of J2.29 (Pin_29)
- net PD3: no longer names the net of J2.32 (Pin_32)
- net PD4: no longer names the net of J2.31 (Pin_31)
- net PD5: no longer names the net of J2.34 (Pin_34)
- net PD6: no longer names the net of J2.33 (Pin_33)
- net PD7: no longer names the net of J2.36 (Pin_36)
- net PD8: no longer names the net of J2.8 (Pin_8)
- net PD9: no longer names the net of J2.7 (Pin_7)
- net PE0: no longer names the net of J2.44 (Pin_44)
- net PE1: no longer names the net of J2.43 (Pin_43)
- net PE10: no longer names the net of J3.18 (Pin_18)
- net PE11: no longer names the net of J3.17 (Pin_17)
- net PE12: no longer names the net of J3.16 (Pin_16)
- net PE13: no longer names the net of J3.15 (Pin_15)
- net PE14: no longer names the net of J3.14 (Pin_14)
- net PE15: no longer names the net of J3.13 (Pin_13)
- net PE2: no longer names the net of J3.44 (Pin_44)
- net PE3: no longer names the net of J3.43 (Pin_43)
- net PE4: no longer names the net of J3.42 (Pin_42)
- net PE5: no longer names the net of J3.41 (Pin_41)
- net PE6: no longer names the net of J3.40 (Pin_40)
- net PE7: no longer names the net of J3.21 (Pin_21)
- net PE8: no longer names the net of J3.20 (Pin_20)
- net PE9: no longer names the net of J3.19 (Pin_19)
- net VDDA: no longer names the net of J3.5 (Pin_5)
- net VREF+: no longer names the net of J3.6 (Pin_6)
Other:
- removed sheet display
- removed sheet ins
- removed sheet power
- added sheet IO (IO.kicad_sch)
- moved on the sheet: H1, H2, H3, H4

Commit message: f
Changed lines of the file:
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@@
 	(text_box "Looking into INS(GPS+IMU) support and Battery Charging and SPI OLED Display support"
 		(exclude_from_sim no)
-		(at 91.44 40.64 0)
+		(at 95.25 55.88 0)
 		(size 35.56 8.89)
 		(margins 0.9525 0.9525 0.9525 0.9525)
